File: hardware/pi-box/pi-box.kicad_sch (KiCad schematic)
At the start: 5 parts, among them J1 Raspberry_Pi_4, J2 RJ45, J3 RJ45

Commit message: Finish the pi-box schematic: clean ERC, verified netlist
Completes the breakout board that replaces the jury-rigged GPIO header.
Zero ERC violations, down from 19 at the first run.

The substance is the two 3.3k pull-ups. With 4.5 m of Cat5 on the bus, SDA's
rise time against the Pi's internal 1.8k is around 400 ns against the 300 ns
Fast-mode allows at 400 kHz, so the bus has been out of spec since the pods
were wired rather than since anything broke. In parallel these give about
1165 ohms, roughly 257 ns, and 2.8 mA of sink — inside what the ADXL345 is
specified to handle.

Also a status LED on GPIO27 through 1k. Driven in software rather than off
the bus, both because anything hung on SDA/SCL costs capacitance the rise
time cannot spare, and because "there is traffic" is the least useful thing
it could report. The failure that started all this was intermittent: the
front pod attached, threw Errno 5 for 25 seconds, then died. An activity
light would have looked healthy throughout.

Netlist verified against the cables as actually built: each signal in its own
twisted pair with a ground return, SDA and SCL never sharing a twist, and
INT1 already run on brown to both pods. The four I2S pins are flagged
no-connect rather than left floating — the stacking header passes them
through mechanically, which is a property of the connector and not of any net
on this sheet.

Ignoring .history/ so the editor's local history stays out of the repo.

Co-Authored-By: Claude Opus 5 <noreply@anthropic.com>
Parts:
- added R2: 3.3k, symbol Device:R
- added R3: 1k, symbol Device:R
- R1: renamed from R3; value R -> 3.3k
Connections:
- net +3.3V: now also R1.1, R2.1
- net GND: now also D1.1 (K)
- net SCL: now also R1.2
- net SDA: now also R2.2
- net at D1.2 (A): now also R3.1
- net at J1.13 (GPIO27/SDIO_DAT3): now also R3.2
- no-connect marks 21 -> 24
Other:
- moved on the sheet: D1, J1, J2, R1

Commit message: Start the pi-box layout: HAT outline and footprints placed
Board outline, mounting holes and header position come from KiCad's own
RaspberryPi-HAT template rather than being drawn by hand — 65 x 56 mm with
radiused corners, four M2.5 holes at 58 x 49 mm, and the 2x20 socket at
+8.37, +4.77 from the top-left corner. Deriving that geometry by measurement
is how a board ends up not fitting.

The socket is on B.Cu at -90 degrees, matching the template. That matters
more than it looks: the female header hangs below the board to mate onto the
Pi's pins, so it is a bottom-side part, and a bottom-side footprint is
mirrored. On the front layer it fabs perfectly and connects SDA to a ground
pin.

Through-hole throughout. Partly for hand-soldering, but mainly because the
two pull-ups may have to come out if the DAC HAT is ever added — that board
brings its own I2C pull-ups, and three sets in parallel would drop the bus
below the 3 mA an ADXL345 is specified to sink. Axials lift with an iron;
0805s do not, on a board bolted into a rack.

Jacks are the Amphenol 54602 horizontal, which is the one plain 8P8C in the
KiCad library. Almost every other horizontal RJ45 there is an Ethernet
magjack with transformers inside, and magnetics do not pass DC, so one of
those would have produced a board that is electrically dead and looks right.

Nothing is placed yet beyond the header.

Co-Authored-By: Claude Opus 5 <noreply@anthropic.com>
Parts:
- D1: footprint (none) -> LED_THT:LED_D3.0mm_Horizontal_O1.27mm_Z10.0mm
- J1: footprint (none) -> Connector_PinSocket_2.54mm:PinSocket_2x20_P2.54mm_Vertical
- J2, J3: footprint (none) -> Connector_RJ:RJ45_Amphenol_54602-x08_Horizontal
- R1, R2, R3: footprint (none) -> Resistor_THT:R_Axial_DIN0207_L6.3mm_D2.5mm_P10.16mm_Horizontal
Changed lines of the file:
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@@
 			)
 		)
-		(property "Footprint" ""
+		(property "Footprint" "LED_THT:LED_D3.0mm_Horizontal_O1.27mm_Z10.0mm"
 			(at 88.9 110.49 0)
 			(hide yes)
@@
 			)
 		)
-		(property "Footprint" ""
+		(property "Footprint" "Connector_RJ:RJ45_Amphenol_54602-x08_Horizontal"
 			(at 55.88 94.615 90)
 			(hide yes)
@@
 			)
 		)
-		(property "Footprint" ""
+		(property "Footprint" "Resistor_THT:R_Axial_DIN0207_L6.3mm_D2.5mm_P10.16mm_Horizontal"
 			(at 49.022 123.19 90)
 			(hide yes)
@@
 			)
 		)
-		(property "Footprint" ""
+		(property "Footprint" "Resistor_THT:R_Axial_DIN0207_L6.3mm_D2.5mm_P10.16mm_Horizontal"
 			(at 57.912 123.19 90)
 			(hide yes)
@@
 			)
 		)
-		(property "Footprint" ""
+		(property "Footprint" "Connector_RJ:RJ45_Amphenol_54602-x08_Horizontal"
 			(at 54.61 62.865 90)
 			(hide yes)
@@
 			)
 		)
-		(property "Footprint" ""
+		(property "Footprint" "Resistor_THT:R_Axial_DIN0207_L6.3mm_D2.5mm_P10.16mm_Horizontal"
 			(at 90.678 102.87 90)
 			(hide yes)
@@
 			)
 		)
-		(property "Footprint" ""
+		(property "Footprint" "Connector_PinSocket_2.54mm:PinSocket_2x20_P2.54mm_Vertical"
 			(at 192.024 123.698 0)
 			(hide yes)
